File: Pico-Breakout.kicad_sch (KiCad schematic)
At the start: 3 parts, among them J101 Conn_01x20, J102 Conn_01x20, U101 Pico

Commit message: Added 3D stacking header
Parts:
- U101: footprint MCU_RaspberryPi_and_Boards:RPi_Pico_TH -> Pico:RPi_Pico_Stacking_TH
Changed lines of the file:
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@@
     (property "Reference" "U101" (id 0) (at 140.97 66.675 0))
     (property "Value" "Pico" (id 1) (at 140.97 69.215 0))
-    (property "Footprint" "MCU_RaspberryPi_and_Boards:RPi_Pico_TH" (id 2) (at 140.97 98.425 90)
+    (property "Footprint" "Pico:RPi_Pico_Stacking_TH" (id 2) (at 140.97 98.425 90)
       (effects (font (size 1.27 1.27)) hide)
     )
@@
     )
     (path "/7e016cea-062f-4f87-855a-68c5d7a4679a"
-      (reference "U101") (unit 1) (value "Pico") (footprint "MCU_RaspberryPi_and_Boards:RPi_Pico_TH")
+      (reference "U101") (unit 1) (value "Pico") (footprint "Pico:RPi_Pico_Stacking_TH")
     )
   )

Commit message: Names streamlined
Parts:
- U101: footprint Pico:RPi_Pico_Stacking_TH -> Pico:RPi_Pico_Stacking_header_TH
Changed lines of the file:
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@@
     (property "Reference" "U101" (id 0) (at 140.97 66.675 0))
     (property "Value" "Pico" (id 1) (at 140.97 69.215 0))
-    (property "Footprint" "Pico:RPi_Pico_Stacking_TH" (id 2) (at 140.97 98.425 90)
+    (property "Footprint" "Pico:RPi_Pico_Stacking_header_TH" (id 2) (at 140.97 98.425 90)
       (effects (font (size 1.27 1.27)) hide)
     )
@@
     )
     (path "/7e016cea-062f-4f87-855a-68c5d7a4679a"
-      (reference "U101") (unit 1) (value "Pico") (footprint "Pico:RPi_Pico_Stacking_TH")
+      (reference "U101") (unit 1) (value "Pico") (footprint "Pico:RPi_Pico_Stacking_header_TH")
     )
   )
